File: pcb/LowPassFilterModule.sch (KiCad schematic (older format))
At the start: 13 parts, among them J1 SMA, J2 CONN_01X04, J3 SMA, J4 CONN_01X04

Commit message: Update for OpenBeacon 2
Parts:
- removed J1, J3: SMA, EtherkitKicadLibrary:SMA-ENDLAUNCH, symbol BNC
- removed J2, J4: CONN_01X04, Socket_Strips:Socket_Strip_Straight_1x04_Pitch2.54mm, symbol CONN_01X04
- added C2, C4, C6: C, Capacitor_SMD:C_0805_2012Metric, symbol EtherkitKicadLibrary:C
- added J1: Conn_01x05, Connector_PinHeader_2.54mm:PinHeader_1x05_P2.54mm_Vertical, symbol Connector_Generic:Conn_01x05
- added J2: Conn_01x04, Connector_PinHeader_2.54mm:PinHeader_1x04_P2.54mm_Vertical, symbol Connector_Generic:Conn_01x04
- C1: footprint Resistors_SMD:R_1206 -> Capacitor_SMD:C_0805_2012Metric; symbol C -> EtherkitKicadLibrary:C
- C3: renamed from C2; footprint Resistors_SMD:R_1206 -> Capacitor_SMD:C_0805_2012Metric; symbol C -> EtherkitKicadLibrary:C
- C5: renamed from C3; footprint Resistors_SMD:R_1206 -> Capacitor_SMD:C_0805_2012Metric; symbol C -> EtherkitKicadLibrary:C
- C7: renamed from C4; footprint Resistors_SMD:R_1206 -> Capacitor_SMD:C_0805_2012Metric; symbol C -> EtherkitKicadLibrary:C
- L1, L2, L3: symbol L-IRONCORE -> EtherkitKicadLibrary:L-IRONCORE
- R1, R2: footprint Resistors_SMD:R_0603 -> Resistor_SMD:R_0603_1608Metric; symbol R -> EtherkitKicadLibrary:R
Connections:
- net GND: now also J1.1 (Pin_1), J1.3 (Pin_3), J1.5 (Pin_5), J2.2 (Pin_2), J2.4 (Pin_4)
- net VCC: now also J2.1 (Pin_1)
- net at C7.1, L3.2: now also C6.1, J2.3 (Pin_3)
- net at C1.1, L1.1: now also C2.2, J1.4 (Pin_4)
- net at C3.1, L1.2, L2.1: now also C2.1, C4.2
- net at C5.1, L2.2, L3.1: now also C4.1, C6.2
- net at R1.2, R2.1: now also J1.2 (Pin_2)
Other:
- note added: "1 uH (T37-2 16T)"
- note added: "1.1 uH (T37-2 17T)"
- note added: "1.2 nF"
- note added: "1.3 nF"
- note added: "1.6 uH (T37-2 20T)"
- note added: "1.8 nF"
- note added: "11 pF"
- note added: "11 uH (FT37-61 14T)"
- note added: "110 pF"
- note added: "12.2 uH (FT37-61 15T)"
- note added: "122 nH (T37-6 6T)"
- note added: "13 pF"
- note added: "130 pF"
- note added: "15 m/12 m/10 m"
- note added: "15 nF"
- note added: "16 pF"
- note added: "160 pF"
- note added: "176 nH (T37-6 8T)"
- note added: "18 nF"
- note added: "18 uH (FT37-61 18T)"
- note added: "195 nH (FT37-61 8T)"
- note added: "2 m/1.25 m"
- note added: "2 nF"
- note added: "2.2 nF"
- note added: "2.4 pF"
- note added: "2.6 uH (FT37-61 7T)"
- note added: "2.9 uH (FT37-61 7T)"
- note added: "20 m/17 m"
- note added: "20 nF"
- note added: "20 pF"
- note added: "200 pF"
- note added: "23 nH (T37-0 6T)"
- note added: "24 nF"
- note added: "240 pF"
- note added: "247 MHz"
- note added: "26 nH (T37-0 6T)"
- note added: "27 nF"
- note added: "287 uH (T37-6 10T)"
- note added: "291 nH (T37-6 10T)"
- note added: "3.9 nF"
- note added: "30 pF"
- note added: "322 nH (T37-6 10T)"
- note added: "33 nF"
- note added: "36 pF"
- note added: "360 pF"
- note added: "38 nH (T37-0 9T)"
- note added: "38 uH (FT37-43 10T)"
- note added: "4.3 nF"
- note added: "4.3 uH (FT37-61 9T)"
- note added: "40 m/30 m"
- note added: "43 uH (FT37-43 11T)"
- note added: "430 pF"
- note added: "470 pF"
- note added: "474 nH (T37-6 13T)"
- note added: "5.1 nF"
- note added: "51 pF"
- note added: "510 pF"
- note added: "520 nH (T37-2 11T)"
- note added: "575 nH (T37-2 12T)"
- note added: "6 m/4 m"
- note added: "6.2 nF"
- note added: "62 pF"
- note added: "62 uH (FT37-43 13T)"
- note added: "68 pF"
- note added: "680 pF"
- note added: "7.5 nF"
- note added: "7.5 pF"
- note added: "75 nH (T37-6 5T)"
- note added: "8.2 nF"
- note added: "80 m/60 m"
- note added: "820 pF"
- note added: "83 uH (T37-6 5T)"
- note added: "846 nH (T37-2 15T)"
- note added: "9.1 nF"
- note added: "9.1 pF"
- note added: "91 pF"
- note added: "Bands"
- note added: "C1"
- note added: "C2"
- note added: "C3"
- note added: "C4"
- note added: "C5"
- note added: "C6"
- note added: "C7"
- note added: "Design: Cauer 0.2 dB ripple, 50 dB stop band, 7th order\n\nSynthesized from the\nARRL Handbook 2014 p11.14 and Table 11.18"
- note added: "L1"
- note added: "L3"
- note removed: "1.04 uH (T37-6 18T)"
- note removed: "1.17 uH (T37-6 19T)"
- note removed: "1.43 uH (T37-2 19T)"
- note removed: "1.61 uH (T37-2 20T)"
- note removed: "1.91 uH (T37-2 22T)"
- note removed: "10 m"
- note removed: "12 m"
- note removed: "12 nF"
- note removed: "148 nH (T37-0 14T)"
- note removed: "15 m"
- note removed: "15.8 MHz"
- note removed: "163 MHz"
- note removed: "166 nH (T37-0 15T)"
- note removed: "17 m"
- note removed: "180 pF"
- note removed: "190 nH (T37-6 7T)"
- note removed: "2 m"
- note removed: "2.19 uH (T37-2 23T)"
- note removed: "2.6 uH (T37-2 25T)"
- note removed: "2.93 uH (T37-2 27T)"
- note removed: "20 m"
- note removed: "21.7 uH (FT37-61 20T)"
- note removed: "215 nH (T37-6 8T)"
- note removed: "220 pF"
- note removed: "23.6 MHz"
- note removed: "24.5 uH (FT37-61 21T)"
- note removed: "27.5 MHz"
- note removed: "3 nF"
- note removed: "30 m"
- note removed: "300 pF"
- note removed: "346 nH (T37-6 10T)"
- note removed: "390 nH (T37-6 11T)"
- note removed: "390 pF"
- note removed: "4 m"
- note removed: "4.4 MHz"
- note removed: "40 m"
- note removed: "415 nH (T37-6 11T)"
- note removed: "469 nH (T37-6 12T)"
- note removed: "485 nH (T37-6 12T)"
- note removed: "5.2 uH (FT37-61 10T)"
- note removed: "5.86 uH (FT37-61 11T)"
- note removed: "547 nH (T37-6 13T)"
- note removed: "560 pF"
- note removed: "571 nH (T37-6 13T)"
- note removed: "6 m"
- note removed: "6.3 nF"
- note removed: "60 MHz"
- note removed: "60 m"
- note removed: "645 nH (T37-6 14T)"
- note removed: "70 nH (T37-0 9T)"
- note removed: "723 nH (T37-6 15T)"
- note removed: "750 pF"
- note removed: "8 MHz"
- note removed: "80 m"
- note removed: "80 nH (T37-0 10T)"
- note removed: "816 nH (T37-6 16T)"
- note removed: "Band"
- note removed: "C1, C4"
- note removed: "C2, C3"
- note removed: "Design: Chebyshev 0.044 dB ripple\n\nSynthesized from the\nARRL Handbook 2014 p11.12 and Table 11.6"
- note removed: "L1, L3"
- moved on the sheet: R1, R2
